File: PBSEQ-D1.kicad_sch (KiCad schematic)
At the start: 19 parts, among them J1 POWER IN, J2 POWER OUT, J3 BUTTON, Q1 AO3401A, Q2 AO3400A, SW1 BUTTON

Commit message: R0.2
* Fixed the diode connection issue. The Cathode was connected to the wrong point.
* Updated `Q1` to AO3415.
* The circuit has been tested and working.
* Updated all 0603 footprints to hand-soldering type for easy soldering.
* Rearranged the silkscreen labels.
* DRC passes.
* Updated BoM.
Parts:
- C1, C2, C3: footprint Capacitor_SMD:C_0603_1608Metric -> Capacitor_SMD:C_0603_1608Metric_Pad1.08x0.95mm_HandSolder
- D2, D3: footprint LED_SMD:LED_0603_1608Metric -> LED_SMD:LED_0603_1608Metric_Pad1.05x0.95mm_HandSolder
- Q1: value AO3401A -> AO3415; MPN AO3401A -> AO3415
- R1, R2, R3, R4, R5, R6, R7: footprint Resistor_SMD:R_0603_1608Metric -> Resistor_SMD:R_0603_1608Metric_Pad0.98x0.95mm_HandSolder
Connections:
- net at C3.2, J3.1 (Pin_1), R1.1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: now also D1.1 (K)
- net at C1.2, C3.1, Q1.1 (G)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: no longer D1.1 (K)
Other:
- moved on the sheet: D1, Q2, R4, R5
